Commit message: add Gazebo colors and remove gravity from propeller

File: bmb_description/urdf/aris.urdf.xacro (robot description, xacro)
@@ -110,13 +110,21 @@
     <gazebo reference="body">
         <gravity>0</gravity>
+        <material>Gazebo/Black</material>
+    </gazebo>
+    <gazebo reference="propeller">
+        <gravity>0</gravity>
+        <material>Gazebo/Green</material>
     </gazebo>
     <gazebo reference="right_aileron">
         <gravity>0</gravity>
+        <material>Gazebo/Gold</material>
     </gazebo>
     <gazebo reference="left_aileron">
         <gravity>0</gravity>
+        <material>Gazebo/Gold</material>
     </gazebo>
     <gazebo reference="elevator">
         <gravity>0</gravity>
+        <material>Gazebo/Gold</material>
     </gazebo>
     <gazebo>

Commit message: add center of mass offset to urdf, documentation

File: bmb_description/urdf/aris.urdf.xacro (robot description, xacro)
@@ -1,4 +1,8 @@
 <?xml version="1.0"?>
 <robot xmlns:xacro="http://www.ros.org/wiki/xacro" name="aris">
+    <!--
+    The meshes are all in the NWU body-relative coordinate system
+    except that the origin is offset from the center of mass
+    -->
     <xacro:property name="infty" value="${1e9}"/>
     <!-- Needs to be large enough so Gazebo doesn't ignore the links/joints -->
@@ -59,4 +63,5 @@
             <inertia ixx="12.327" ixy="-3.07" ixz="0.739"
                      iyy="1.711" iyz="-2.789" izz="12.659"/>
+            <origin xyz="-0.12195 0.00111 0.06595" rpy="0 0 0"/>
         </inertial>
         <collision>

Commit message: remove off-diagonal elements from inertia matrix

File: bmb_description/urdf/aris.urdf.xacro (robot description, xacro)
@@ -61,7 +61,6 @@
         <inertial>
             <mass value="3.3"/>
-            <inertia ixx="12.327" ixy="-3.07" ixz="0.739"
-                     iyy="1.711" iyz="-2.789" izz="12.659"/>
-            <origin xyz="-0.12195 0.00111 0.06595" rpy="0 0 0"/>
+            <inertia ixx="12.327" ixy="0" ixz="0"
+                     iyy="1.711" iyz="0" izz="12.659"/>
         </inertial>
         <collision>
